File: laser-assembly/LED-holder.kicad_sch (KiCad schematic)
At the start: 7 parts, among them J1 Conn_01x01_Pin, J2 Conn_01x01_Pin, J3 Conn_01x01_Pin, SW1 SW_SPDT

Commit message: fixed bom comment and video
Parts:
- D1: Comment Mount on the front with the full pun length -> Mount on the front with the full pin length
Changed lines of the file:
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@@
 			)
 		)
-		(property "Comment" "Mount on the front with the full pun length"
+		(property "Comment" "Mount on the front with the full pin length"
 			(at 149.86 55.88 90)
 			(hide yes)
